File: cresk_choc/cresk_choc.kicad_sch (KiCad schematic)
At the start: 21 parts, among them J1 TRRS, J2 BATTERY, SW1 SW_Push, SW10 SW_Push, SW11 SW_Push, SW12 SW_Push, SW13 SW_Push, SW14 SW_Push, SW15 SW_Push, SW16 SW_Push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

Commit message: cresk_choc: finish routing
Parts:
- SW1, SW10, SW11, SW16, SW17, SW5, SW6: footprint cresk:Kailh_Choc_Socket_Reversible_Plain_Alt -> cresk:Kailh_Choc_Reversible
- SW12, SW13, SW14, SW15, SW2, SW3, SW4, SW7, SW8, SW9: footprint cresk:Kailh_Choc_Socket_Reversible_Plain -> cresk:Kailh_Choc_Reversible
Connections:
- net GND: now also SW1.2, SW11.2, SW6.2; no longer SW1.1, SW11.1, SW6.1
- net sw1: now also SW1.1, U1.8; no longer SW1.2, U1.11
- net sw10: now also U1.11; no longer U1.10
- net sw11: now also SW11.1; no longer SW11.2
- net sw2: now also U1.7; no longer U1.20
- net sw3: now also U1.6; no longer U1.1 (TX)
- net sw5: now also U1.1 (TX); no longer U1.6
- net sw6: now also SW6.1, U1.20; no longer SW6.2, U1.12
- net sw7: now also U1.12; no longer U1.7
- net sw8: now also U1.9; no longer U1.8
- net sw9: now also U1.10; no longer U1.9
Other:
- moved on the sheet: SW1, SW11, SW6
